File: 16F676-mppt.kicad_pcb (KiCad board)
At the start: 2 copper layers, 96.5 x 87.6 mm, 54 parts, among them J1 S+, J2 S-, J3 VB+, J4 VB-, Q1 BUK9511-55A127, Q2 BUK9511-55A127, Q3 2N2222A, Q4 2N2222A, Q5 2N2907A, SW1 Write OP-AMP DIFF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

Commit message: Update PCB Layout.
Parts:
- removed R11: 100k, Resistors_THT:R_Axial_DIN0309_L9.0mm_D3.2mm_P12.70mm_Horizontal
- D3: value 1N4001 -> 1N4148
- moved R1 5.84 mm to (36.8, 82.3)
- moved R15 3.83 mm to (31.7, 82.3)
Connections:
- C5 pad 1: Net-(C5-Pad1) -> /PV-Current
- U3 pad 13: Net-(C5-Pad1) -> /PV-Current
Routing:
- net /PV-Current: track 22.2 -> 100.8 mm, vias 0 -> 1
- net Net-(C5-Pad1): track 55.3 -> 0.00 mm
- net GND: track 380.0 -> 358.2 mm
- net Net-(R1-Pad2): track 47.7 -> 31.3 mm
- net Net-(R3-Pad1): track 35.1 -> 32.5 mm
- net Net-(R4-Pad1): track 27.6 -> 28.8 mm

Commit message: update PCB.
Parts:
- removed R17: 1k, Resistors_THT:R_Axial_DIN0309_L9.0mm_D3.2mm_P2.54mm_Vertical
Connections:
- Q4 pad 1: Net-(Q4-Pad1) -> Net-(Q2-Pad1)
- Q5 pad 1: Net-(Q4-Pad1) -> Net-(Q2-Pad1)
Routing:
- net Net-(Q4-Pad1): track 13.8 -> 0.00 mm
- net Net-(Q2-Pad1): track 8.44 -> 11.3 mm
Changed lines of the file:
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@@
     (thickness 1.6)
     (drawings 4)
-    (tracks 298)
+    (tracks 296)
     (zones 0)
-    (modules 53)
-    (nets 35)
+    (modules 52)
+    (nets 34)
   )
   (page User 150.012 170.002)
@@
   )
   (setup
-    (last_trace_width 1)
+    (last_trace_width 1.5)
     (user_trace_width 0.5)
     (user_trace_width 1)
@@
   (net 32 GND)
   (net 33 VDD)
-  (net 34 "Net-(Q4-Pad1)")
   (net_class Default "This is the default net class."
     (clearance 0.2)
@@
     (add_net "Net-(Q3-Pad2)")
     (add_net "Net-(Q3-Pad3)")
-    (add_net "Net-(Q4-Pad1)")
     (add_net "Net-(Q4-Pad2)")
     (add_net "Net-(R1-Pad2)")
@@
     (pad 1 thru_hole circle (at 0 0) (size 5 5) (drill 2.5) (layers *.Cu *.Mask))
   )
-  (module Resistors_THT:R_Axial_DIN0309_L9.0mm_D3.2mm_P2.54mm_Vertical (layer F.Cu)
-    (at 76.18476 19.31416 90)
-    (descr "Resistor, Axial_DIN0309 series, Axial, Vertical, pin pitch=2.54mm, 0.5W = 1/2W, length*diameter=9*3.2mm^2, http://cdn-reichelt.de/documents/datenblatt/B400/1_4W%23YAG.pdf")
-    (tags "Resistor Axial_DIN0309 series Axial Vertical pin pitch 2.54mm 0.5W = 1/2W length 9mm diameter 3.2mm")
-    (fp_text reference R17 (at 1.74244 -2.70256 90) (layer F.SilkS)
-      (effects (font (size 1 1) (thickness 0.15)))
-    )
-    (fp_text value 1k (at 1.27 2.66 90) (layer F.Fab)
-      (effects (font (size 1 1) (thickness 0.15)))
-    )
-    (fp_arc (start 0 0) (end 1.45451 -0.8) (angle -302.4) (layer F.SilkS) (width 0.12))
-    (fp_circle (center 0 0) (end 1.6 0) (layer F.Fab) (width 0.1))
-    (fp_line (start 0 0) (end 2.54 0) (layer F.Fab) (width 0.1))
-    (fp_line (start -1.95 -1.95) (end -1.95 1.95) (layer F.CrtYd) (width 0.05))
-    (fp_line (start -1.95 1.95) (end 3.65 1.95) (layer F.CrtYd) (width 0.05))
-    (fp_line (start 3.65 1.95) (end 3.65 -1.95) (layer F.CrtYd) (width 0.05))
-    (fp_line (start 3.65 -1.95) (end -1.95 -1.95) (layer F.CrtYd) (width 0.05))
-    (pad 1 thru_hole circle (at 0 0 90) (size 1.6 1.6) (drill 0.8) (layers *.Cu *.Mask)
-      (net 34 "Net-(Q4-Pad1)"))
-    (pad 2 thru_hole oval (at 2.54 0 90) (size 1.6 1.6) (drill 0.8) (layers *.Cu *.Mask)
-      (net 11 "Net-(Q2-Pad1)"))
-    (model ${KISYS3DMOD}/Resistors_THT.3dshapes/R_Axial_DIN0309_L9.0mm_D3.2mm_P2.54mm_Vertical.wrl
-      (at (xyz 0 0 0))
-      (scale (xyz 0.393701 0.393701 0.393701))
-      (rotate (xyz 0 0 0))
-    )
-  )
   (module Housings_DIP:DIP-8_W7.62mm placed (layer F.Cu)
     (at 44.958 55.88)
@@
       (net 1 "Net-(C2-Pad1)"))
     (pad 1 thru_hole rect (at 0 0) (size 1.52 1.52) (drill 0.8) (layers *.Cu *.Mask)
-      (net 34 "Net-(Q4-Pad1)"))
+      (net 11 "Net-(Q2-Pad1)"))
     (model ${KISYS3DMOD}/TO_SOT_Packages_THT.3dshapes/TO-92_Inline_Wide.wrl
       (offset (xyz 2.539999961853027 0 0))
@@
       (net 2 "Net-(C2-Pad2)"))
     (pad 1 thru_hole rect (at 0 0) (size 1.52 1.52) (drill 0.8) (layers *.Cu *.Mask)
-      (net 34 "Net-(Q4-Pad1)"))
+      (net 11 "Net-(Q2-Pad1)"))
     (model ${KISYS3DMOD}/TO_SOT_Packages_THT.3dshapes/TO-92_Inline_Wide.wrl
       (offset (xyz 2.539999961853027 0 0))
@@
   (segment (start 49.784 88.646) (end 60.706 88.646) (width 1) (layer F.Cu) (net 10))
   (segment (start 47.244 91.186) (end 47.244 93.726) (width 1) (layer F.Cu) (net 10))
-  (segment (start 81.89976 16.77416) (end 76.18476 16.77416) (width 1.5) (layer B.Cu) (net 11))
-  (segment (start 83.82508 18.69948) (end 81.89976 16.77416) (width 1.5) (layer B.Cu) (net 11))
   (segment (start 77.978 41.148) (end 77.978 30.988) (width 1) (layer F.Cu) (net 12))
   (segment (start 66.802 52.324) (end 77.978 41.148) (width 1) (layer F.Cu) (net 12))
@@
   (segment (start 23.622 30.988) (end 23.622 31.242) (width 3) (layer B.Cu) (net 33))
   (segment (start 23.622 26.162) (end 23.622 18.542) (width 3) (layer B.Cu) (net 33))
-  (segment (start 77.98816 19.31416) (end 82.55 23.876) (width 1.5) (layer B.Cu) (net 34))
-  (segment (start 76.18476 19.31416) (end 77.98816 19.31416) (width 1.5) (layer B.Cu) (net 34))
-  (segment (start 82.55 23.876) (end 88.138 23.876) (width 1.5) (layer B.Cu) (net 34))
+  (segment (start 82.55 23.876) (end 88.138 23.876) (width 1.5) (layer B.Cu) (net 11))
+  (segment (start 83.82508 22.60092) (end 82.55 23.876) (width 1.5) (layer B.Cu) (net 11))
+  (segment (start 83.82508 18.69948) (end 83.82508 22.60092) (width 1.5) (layer B.Cu) (net 11))
   (zone (net 0) (net_name "") (layer B.Cu) (hatch edge 0.508)
     (connect_pads (clearance 0.508))

Commit message: update pcb.
Parts:
- removed C6: 10u, Capacitors_THT:CP_Radial_D12.5mm_P5.00mm
- added Q6: 2N2222A, TO_SOT_Packages_THT:TO-92_Inline_Wide, F.Cu at (36.6, 56.5)
- added Q7: 2N2222A, TO_SOT_Packages_THT:TO-92_Inline_Wide, F.Cu at (31.0, 51.4)
- R15: value 10k -> 2.2k
- moved R8 13.7 mm to (24.5, 59.6)
- moved U1 9.62 mm to (28.4, 47.7)
Routing:
- net Net-(R8-Pad2): track 70.4 -> 28.9 mm
- net /PV-Voltage: track 7.46 -> 30.6 mm
- net Net-(Q6-Pad2): track 0.00 -> 10.7 mm
- net Net-(D5-Pad1): track 17.3 -> 7.36 mm
- net GND: track 358.2 -> 350.6 mm
- net Net-(Q3-Pad2): track 34.6 -> 31.1 mm

Commit message: update PCB.
Parts:
- added R11: 10k, Resistors_THT:R_Axial_DIN0309_L9.0mm_D3.2mm_P12.70mm_Horizontal, F.Cu at (58.3, 36.4)
- moved C4 6.95 mm to (65.1, 38.7)
Routing:
- net GND: track 350.6 -> 339.9 mm
- net /BootStrap: track 104.3 -> 113.1 mm
- net Net-(R11-Pad2): track 10.6 -> 17.6 mm
