File: 16F676-mppt.kicad_sch (KiCad schematic)
At the start: 54 parts, among them J1 S+, J2 S-, J3 VB+, J4 VB-, Q1 BUK9511-55A127, Q2 BUK9511-55A127, Q3 2N2222A, Q4 2N2222A, Q5 2N2907A, Q6 2N2222A, Q7 2N2222A, SW1 Write OP-AMP DIFF, U1 LM7805_TO220, U2 LM358N, U3 16F676, Y1 12MHz

Commit message: Change capacitors.
Parts:
- removed C2: 4.7uF 50v, Capacitor_THT:CP_Radial_D8.0mm_P2.50mm, symbol Device:CP
- removed C5: 10u, Capacitor_THT:CP_Radial_D8.0mm_P2.50mm, symbol Device:CP
- added C2: 1u, symbol Device:C
- added C5: 10u, symbol Device:C
Connections:
- net < 3.6V: now also C5.1
- net BootStrap: now also C2.1
- net GND: now also C5.2
- net at D1.2 (A), D10.2 (A), D12.2 (A)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: now also C2.2

Commit message: Update capacitor footprint.
Parts:
- C2, C5: footprint (none) -> Capacitors_THT:C_Disc_D12.5mm_W5.0mm_P7.50mm
Changed lines of the file:
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@@
 			)
 		)
-		(property "Footprint" ""
+		(property "Footprint" "Capacitors_THT:C_Disc_D12.5mm_W5.0mm_P7.50mm"
 			(at 191.4652 73.66 0)
 			(hide yes)
@@
 			)
 		)
-		(property "Footprint" ""
+		(property "Footprint" "Capacitors_THT:C_Disc_D12.5mm_W5.0mm_P7.50mm"
 			(at 169.8752 128.27 0)
 			(hide yes)
